File: HostSide.kicad_sch (KiCad schematic)
At the start: 16 parts, among them J2 53014-1010, J3 Push_In_2.54mm_Terminal_141V-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, Q1 NTK3134NT1G, Q2 NTK3134NT1G, Q3 NTK3134NT1G, Q4 NTK3134NT1G, U3 74HC4049

Commit message: init to 0.2
Parts:
- renumbered C10 to C14, C11 to C15, C12 to C16, J2 to J1, J3 to J2
