File: LambdaTail-HW.kicad_pcb (KiCad board)
At the start: 2 copper layers, 55 x 55 mm, 71 parts, among them J1 DC JACK - (5.0x2.0 pi), J2 53014-1010, J3 Push_In_2.54mm_Terminal_141V-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, J4 53014-1010, J5 Push_In_2.54mm_Terminal_141V-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, Q1 NTK3134NT1G, Q2 NTK3134NT1G, Q3 NTK3134NT1G, Q4 NTK3134NT1G, Q5 NTK3134NT1G, Q6 NTK3134NT1G, U1 ESP32-WROOM-32E (4MB), U2 RT8259GJ6, U3 74HC4049

Commit message: init to 0.2
Parts:
- removed the C18 at (60.5, 69.6)
- removed the D3 at (55.9, 77.0)
- removed the J1 at (55.0, 86.7)
- removed the R9 at (52.3, 64.9)
- added C10: 100nF, Capacitor_SMD:C_0402_1005Metric, F.Cu at (130.4, 58.5)
- added C11: 100nF, Capacitor_SMD:C_0402_1005Metric, F.Cu at (125.8, 53.2)
- added C12: 22uF, Capacitor_SMD:C_0805_2012Metric, F.Cu at (119.3, 48.3)
- added C13: 22uF, Capacitor_SMD:C_0805_2012Metric, F.Cu at (119.3, 50.5)
- added D1: B260, Diode_SMD:D_SMB, F.Cu at (125.5, 70.9)
- added L1: LQM21PN1R5MC0D, Inductor_SMD:L_0805_2012Metric, F.Cu at (130.3, 62.5)
- added R6: 100.0 mOhm, Resistor_SMD:R_0402_1005Metric, F.Cu at (128.6, 60.8)
- C6, C9: value 100nF -> 10uF; footprint Capacitor_SMD:C_0402_1005Metric -> Capacitor_SMD:C_0805_2012Metric
- C7: value 10nF -> 10uF; footprint Capacitor_SMD:C_0402_1005Metric -> Capacitor_SMD:C_0805_2012Metric
- C8: value 22uF -> Tantal 3.3uF 20V; footprint Capacitor_SMD:C_0805_2012Metric -> Capacitor_Tantalum_SMD:CP_EIA-3216-18_Kemet-A
- L2: renamed from L1; value VLS6045EX-4R7M -> ASPI-6045S-120M
- R8: value 16k -> 62k
- U2: value RT8259GJ6 -> LMR50410X; footprint Package_TO_SOT_SMD:TSOT-23-6 -> Package_TO_SOT_SMD:SOT-23-6
- moved C6 75.6 mm to (127.5, 65.2)
- moved C5 73.9 mm to (127.5, 67.2)
- moved U2 73.4 mm to (127.1, 55.6), turned to 0 degrees
- moved R8 70.5 mm to (122.1, 58.0), turned to -90 degrees
- moved C7 70.3 mm to (127.5, 63.2), turned to 180 degrees
- moved R7 70.2 mm to (123.8, 58.0), turned to 90 degrees
- moved L2 70.2 mm to (125.7, 48.8), turned to 180 degrees
- moved C9 63.0 mm to (127.4, 58.5), turned to 180 degrees
- moved C8 62.3 mm to (125.4, 60.8), turned to 180 degrees
- renumbered C10 to C14, C11 to C15, C12 to C16, C13 to C17, C14 to C18, C15 to C19, C16 to C20, C17 to C21, C19 to C22, C20 to C23, D1 to D2, D2 to D3, J2 to J1, J3 to J2, J4 to J3, J5 to J4, R6 to R9
Connections:
- C5 pad 1: +12V -> /Power/LIMITED_+12V
- C6 pad 1: /Power/PWR_EN -> /Power/LIMITED_+12V
- C7 pad 1: /Power/PWR_BOOT -> /Power/LIMITED_+12V
- C7 pad 2: /Power/PWR_PHASE -> GND
- C8 pad 1: +3V3 -> Net-(C8-Pad1)
- C9 pad 1: +3V3 -> /Power/FILTERED_+12V
- D2 pad 1: +12V -> (no net)
- D2 pad 2: GND -> (no net)
- J1 pad 7: unconnected-(J2-Pad7) -> (no net)
- J3 pad 7: unconnected-(J4-Pad7) -> (no net)
- L2 pad 1: /Power/PWR_PHASE -> /Power/PWR_SW
- R7 pad 1: +3V3 -> /Power/PWR_FB
- R7 pad 2: /Power/PWR_FB -> +3V3
- R8 pad 1: /Power/PWR_FB -> +3V3
- R8 pad 2: Net-(R8-Pad2) -> GND
- U2 pad 1: /Power/PWR_BOOT -> /Power/PWR_CB
- U2 pad 4: /Power/PWR_EN -> /Power/FILTERED_+12V
- U2 pad 5: +12V -> /Power/FILTERED_+12V
- U2 pad 6: /Power/PWR_PHASE -> /Power/PWR_SW
Routing:
- net /Power/PWR_SW: track 0.00 -> 10.5 mm
- net /Power/PWR_PHASE: track 6.83 -> 0.00 mm
- net (no net): track 0.00 -> 4.48 mm
- net /Power/PWR_EN: track 1.54 -> 0.00 mm
- net Net-(R8-Pad2): track 1.49 -> 0.00 mm
- net /Power/PWR_BOOT: track 1.45 -> 0.00 mm
- net +12V: vias 8 -> 7
- net GND: vias 222 -> 219
- added copper zone on F.Cu, net (none)
- removed copper zone on F.Cu, net /Power/PWR_PHASE
