File: VendSide.kicad_sch (KiCad schematic)
At the start: 23 parts, among them J4 53014-1010, J5 Push_In_2.54mm_Terminal_141V-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, Q5 NTK3134NT1G, Q6 NTK3134NT1G, U3 74HC4049

Commit message: init to 0.2
Parts:
- removed C18: 100nF, Capacitor_SMD:C_0402_1005Metric, symbol Device:C
- renumbered C13 to C17, C14 to C18, C15 to C19, C16 to C20, C17 to C21, C19 to C22, C20 to C23, J4 to J3, J5 to J4
